Commit message: Update src/quadcopter/urdf/Quadcopter.urdf
The joint limits for continuous joints have incorrect values. For continuous joints, lower and upper limits should not be set to 0, as this would prevent any rotation. Either remove the limit element entirely for truly continuous rotation, or set appropriate non-zero limits if rotation should be constrained.

Co-authored-by: Copilot <175728472+Copilot@users.noreply.github.com>

File: src/quadcopter/urdf/Quadcopter.urdf (robot description, URDF)
Before this commit: robot quadcopter, 6 links, 5 joints
Joints:
- joint propeller_1: limit lower=0 upper=0 effort=10 velocity=1000 -> effort=10 velocity=1000
