Commit message: Add ROS2 control and sensor integration for quadcopter
Introduces ROS2 control configuration and controllers for quadcopter propellers, adds IMU and camera sensor integration, and updates the URDF with a dummy root link to resolve KDL warnings. Launch file is updated to load controllers and bridges for sensor topics. Documentation is expanded with sensor activation instructions and available topics.

File: src/quadcopter/urdf/Quadcopter.urdf (robot description, URDF)
Before this commit: robot quadcopter, 6 links, 5 joints
Links:
- added link base_footprint
- link base_link: mass 0.13344 -> 1.0
Joints:
- added joint base_footprint_to_base: type fixed, parent base_footprint, child base_link, origin xyz=0 0 0 rpy=0 0 0
- joint propeller_2: limit lower=0 upper=0 effort=10 velocity=1000 -> effort=10 velocity=1000
- joint propeller_3: limit lower=0 upper=0 effort=10 velocity=1000 -> effort=10 velocity=1000
- joint propeller_4: limit lower=0 upper=0 effort=10 velocity=1000 -> effort=10 velocity=1000

Commit message: Add simple joint state publisher and improve quadcopter URDF
Introduced a custom simple_joint_state_publisher.py node and integrated it into the Gazebo launch file, replacing the previous joint state bridge. Added installation rules for the new script. Enhanced the Quadcopter.urdf with additional links (IMU, GPS, camera, battery, landing gear), improved inertial and collision properties, and updated Gazebo plugin configurations for better simulation compatibility. Added a robot_desc.yaml for robot_state_publisher configuration.

File: src/quadcopter/urdf/Quadcopter.urdf (robot description, URDF)
Before this commit: robot quadcopter, 7 links, 6 joints
Links:
- added link battery_link, mass 0.2; collision box size=0.08 0.04 0.02; visual box size=0.08 0.04 0.02
- added link camera_optical_link
- added link gps_link, mass 0.001; visual cylinder length=0.005 radius=0.01
- added link imu_link, mass 0.001; visual box size=0.01 0.01 0.005
- added link landing_gear_fl, mass 0.001; collision sphere radius=0.01; visual sphere radius=0.01
- added link landing_gear_fr, mass 0.001; collision sphere radius=0.01; visual sphere radius=0.01
- added link landing_gear_rl, mass 0.001; collision sphere radius=0.01; visual sphere radius=0.01
- added link landing_gear_rr, mass 0.001; collision sphere radius=0.01; visual sphere radius=0.01
- link base_link: mass 1.0 -> 0.8; geometry collision box size=0.25 0.25 0.05; visual mesh filename=package://quadcopter/meshes/base_link.STL
- link link_camera: geometry collision box size=0.02 0.04 0.02; visual mesh filename=package://quadcopter/meshes/link_camera.STL
- link link_propeller_1: mass 0.0024223 -> 0.005; geometry collision cylinder length=0.01 radius=0.1; visual mesh filename=package://quadcopter/meshes/link_propeller_1.STL
- link link_propeller_2: mass 0.0024223 -> 0.005; geometry collision cylinder length=0.01 radius=0.1; visual mesh filename=package://quadcopter/meshes/link_propeller_2.STL
- link link_propeller_3: mass 0.0024223 -> 0.005; geometry collision cylinder length=0.01 radius=0.1; visual mesh filename=package://quadcopter/meshes/link_propeller_3.STL
- link link_propeller_4: mass 0.0024223 -> 0.005; geometry collision cylinder length=0.01 radius=0.1; visual mesh filename=package://quadcopter/meshes/link_propeller_4.STL
Joints:
- added joint battery_joint: type fixed, parent base_link, child battery_link, origin xyz=0 0 -0.02 rpy=0 0 0
- added joint camera_optical_joint: type fixed, parent link_camera, child camera_optical_link, origin xyz=0 0 0 rpy=-1.5708 0 -1.5708
- added joint gps_joint: type fixed, parent base_link, child gps_link, origin xyz=0 0 0.03 rpy=0 0 0
- added joint imu_joint: type fixed, parent base_link, child imu_link, origin xyz=0 0 0 rpy=0 0 0
- added joint landing_gear_fl_joint: type fixed, parent base_link, child landing_gear_fl, origin xyz=-0.08 0.08 -0.04 rpy=0 0 0
- added joint landing_gear_fr_joint: type fixed, parent base_link, child landing_gear_fr, origin xyz=0.08 0.08 -0.04 rpy=0 0 0
- added joint landing_gear_rl_joint: type fixed, parent base_link, child landing_gear_rl, origin xyz=-0.08 -0.08 -0.04 rpy=0 0 0
- added joint landing_gear_rr_joint: type fixed, parent base_link, child landing_gear_rr, origin xyz=0.08 -0.08 -0.04 rpy=0 0 0
- joint base_footprint_to_base: origin xyz=0 0 0 rpy=0 0 0 -> xyz=0 0 0.05 rpy=0 0 0
- joint propeller_1: limit effort=10 velocity=1000 -> effort=10 velocity=2000
- joint propeller_2: limit effort=10 velocity=1000 -> effort=10 velocity=2000
- joint propeller_3: limit effort=10 velocity=1000 -> effort=10 velocity=2000
- joint propeller_4: limit effort=10 velocity=1000 -> effort=10 velocity=2000
